File: servo_beunboard.kicad_sch (KiCad schematic)
At the start: 15 parts, among them J1 ANGLE_SENSOR, J2 SERVO_INPUT, M1 Motor_DC, U1 DRV8212, U2 MT6701, U6 SPX5205M5-L-3.3

Commit message: v1
Parts:
- C3: value BULK -> 22uF; LCSC C15850 -> C45783
- H1, H2: footprint (none) -> servo-hacking:JLC_ToolingHole; now left out of the parts list
Other:
- title: (none) -> Servo Controller
Changed lines of the file:
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@@
 (kicad_sch (version 20230121) (generator eeschema)
   (paper "A4")
+  (title_block
+    (title "Servo Controller")
+    (date "2023-05-01")
+    (rev "v1")
+  )
   (junction (at 161.29 45.72) (diameter 0) (color 0 0 0 0)
   )
@@
   )
   (symbol (lib_id "Mechanical:MountingHole") (at 254 146.05 0) (unit 1)
-    (in_bom yes) (on_board yes) (dnp no) (fields_autoplaced)
+    (in_bom no) (on_board yes) (dnp no) (fields_autoplaced)
     (property "Reference" "H1" (at 256.54 145.415 0)
       (effects (font (size 1.27 1.27)) (justify left))
@@
       (effects (font (size 1.27 1.27)) (justify left))
     )
-    (property "Footprint" "" (at 254 146.05 0)
+    (property "Footprint" "servo-hacking:JLC_ToolingHole" (at 254 146.05 0)
       (effects (font (size 1.27 1.27)) hide)
     )
@@
       (effects (font (size 1.27 1.27)) (justify right))
     )
-    (property "Value" "BULK" (at 69.85 55.245 0)
+    (property "Value" "22uF" (at 69.85 55.245 0)
       (effects (font (size 1.27 1.27)) (justify right))
     )
@@
       (effects (font (size 1.27 1.27)) hide)
     )
-    (property "LCSC" "C15850" (at 66.04 53.34 0)
+    (property "LCSC" "C45783" (at 66.04 53.34 0)
       (effects (font (size 1.27 1.27)) hide)
     )
@@
   )
   (symbol (lib_id "Mechanical:MountingHole") (at 254 154.94 0) (unit 1)
-    (in_bom yes) (on_board yes) (dnp no) (fields_autoplaced)
+    (in_bom no) (on_board yes) (dnp no) (fields_autoplaced)
     (property "Reference" "H2" (at 256.54 154.305 0)
       (effects (font (size 1.27 1.27)) (justify left))
@@
       (effects (font (size 1.27 1.27)) (justify left))
     )
-    (property "Footprint" "" (at 254 154.94 0)
-      (effects (font (size 1.27 1.27)) hide)
-    )
+    (property "Footprint" "servo-hacking:JLC_ToolingHole" (at 254 154.94 0)
+      (effects (font (size 1.27 1.27)) hide)
+    )

Commit message: Change LDO JLC part
Parts:
- added C8: 1uF, Capacitor_SMD:C_0603_1608Metric_Pad1.08x0.95mm_HandSolder, symbol Device:C_Small
- U1: value DRV8212 -> DRV8212DSG
- U6: LCSC C157628 -> C2843766
Connections:
- net GND: now also C8.2
- net VCC: now also C8.1
Changed lines of the file:
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@@
   (junction (at 66.04 49.53) (diameter 0) (color 0 0 0 0)
+  )
+  (junction (at 152.4 45.72) (diameter 0) (color 0 0 0 0)
   )
   (no_connect (at 205.74 48.26))
@@
     (stroke (width 0) (type default))
   )
-  (polyline (pts (xy 148.59 76.2) (xy 256.54 76.2))
+  (polyline (pts (xy 140.97 76.2) (xy 256.54 76.2))
     (stroke (width 0) (type default))
   )
@@
     (stroke (width 0) (type default))
   )
+  (wire (pts (xy 161.29 45.72) (xy 152.4 45.72))
+    (stroke (width 0) (type default))
+  )
   (wire (pts (xy 67.31 128.27) (xy 69.85 128.27))
     (stroke (width 0) (type default))
@@
     (stroke (width 0) (type default))
   )
-  (wire (pts (xy 161.29 41.91) (xy 161.29 45.72))
+  (wire (pts (xy 152.4 41.91) (xy 152.4 45.72))
     (stroke (width 0) (type default))
   )
@@
     (stroke (width 0) (type default))
   )
-  (polyline (pts (xy 148.59 25.4) (xy 256.54 25.4))
+  (wire (pts (xy 152.4 52.07) (xy 152.4 57.15))
+    (stroke (width 0) (type default))
+  )
+  (polyline (pts (xy 140.97 25.4) (xy 256.54 25.4))
     (stroke (width 0) (type default))
   )
@@
     (stroke (width 0) (type default))
   )
-  (polyline (pts (xy 148.59 25.4) (xy 148.59 76.2))
+  (polyline (pts (xy 140.97 25.4) (xy 140.97 76.2))
     (stroke (width 0) (type default))
   )
@@
   )
   (wire (pts (xy 99.06 128.27) (xy 93.98 128.27))
+    (stroke (width 0) (type default))
+  )
+  (wire (pts (xy 152.4 45.72) (xy 152.4 46.99))
     (stroke (width 0) (type default))
   )
@@
     (effects (font (size 1.27 1.27)) (justify left bottom))
   )
-  (text "Encoder + LDO" (at 152.4 74.93 0)
+  (text "Encoder + LDO" (at 142.24 74.93 0)
     (effects (font (size 1.27 1.27)) (justify left bottom))
   )
@@
     )
   )
-  (symbol (lib_id "power:VCC") (at 161.29 41.91 0) (unit 1)
-    (in_bom yes) (on_board yes) (dnp no) (fields_autoplaced)
-    (property "Reference" "#PWR01" (at 161.29 45.72 0)
-      (effects (font (size 1.27 1.27)) hide)
-    )
-    (property "Value" "VCC" (at 161.29 38.1 0)
-      (effects (font (size 1.27 1.27)))
-    )
-    (property "Footprint" "" (at 161.29 41.91 0)
-      (effects (font (size 1.27 1.27)) hide)
-    )
-    (property "Datasheet" "" (at 161.29 41.91 0)
+  (symbol (lib_id "power:VCC") (at 152.4 41.91 0) (unit 1)
+    (in_bom yes) (on_board yes) (dnp no) (fields_autoplaced)
+    (property "Reference" "#PWR01" (at 152.4 45.72 0)
+      (effects (font (size 1.27 1.27)) hide)
+    )
+    (property "Value" "VCC" (at 152.4 38.1 0)
+      (effects (font (size 1.27 1.27)))
+    )
+    (property "Footprint" "" (at 152.4 41.91 0)
+      (effects (font (size 1.27 1.27)) hide)
+    )
+    (property "Datasheet" "" (at 152.4 41.91 0)
       (effects (font (size 1.27 1.27)) hide)
     )
@@
       (effects (font (size 1.27 1.27)) hide)
     )
-    (property "LCSC" "C157628" (at 176.53 46.99 0)
+    (property "LCSC" "C2843766" (at 176.53 46.99 0)
       (effects (font (size 1.27 1.27)) hide)
     )
@@
         (path "/e63e39d7-6ac0-4ffd-8aa3-1841a4541b55/49e00748-0bf6-4cb0-8f84-201c3846ab68"
           (reference "#PWR080") (unit 1)
+        )
+      )
+    )
+  )
+  (symbol (lib_id "power:GND") (at 152.4 57.15 0) (unit 1)
+    (in_bom yes) (on_board yes) (dnp no) (fields_autoplaced)
+    (property "Reference" "#PWR08" (at 152.4 63.5 0)
+      (effects (font (size 1.27 1.27)) hide)
+    )
+    (property "Value" "GND" (at 152.4 62.23 0)
+      (effects (font (size 1.27 1.27)))
+    )
+    (property "Footprint" "" (at 152.4 57.15 0)
+      (effects (font (size 1.27 1.27)) hide)
+    )
+    (property "Datasheet" "" (at 152.4 57.15 0)
+      (effects (font (size 1.27 1.27)) hide)
+    )
+    (pin "1")
+    (instances
+      (project "servo_beunboard"
+        (path "/bf2cf965-926d-44f9-b138-29152ff88b89"
+          (reference "#PWR08") (unit 1)
         )
       )
@@
     )
   )
+  (symbol (lib_id "Device:C_Small") (at 152.4 49.53 0) (unit 1)
+    (in_bom yes) (on_board yes) (dnp no)
+    (property "Reference" "C8" (at 146.05 48.26 0)
+      (effects (font (size 1.27 1.27)) (justify left))
+    )
+    (property "Value" "1uF" (at 146.05 50.8 0)
+      (effects (font (size 1.27 1.27)) (justify left))
+    )
+    (property "Footprint" "Capacitor_SMD:C_0603_1608Metric_Pad1.08x0.95mm_HandSolder" (at 152.4 49.53 0)
+      (effects (font (size 1.27 1.27)) hide)
+    )
+    (property "Datasheet" "~" (at 152.4 49.53 0)
+      (effects (font (size 1.27 1.27)) hide)
+    )
+    (property "LCSC" "C15849" (at 152.4 49.53 0)
+      (effects (font (size 1.27 1.27)) hide)
+    )
+    (pin "1")
+    (pin "2")
+    (instances
+      (project "servo_beunboard"
+        (path "/bf2cf965-926d-44f9-b138-29152ff88b89"
+          (reference "C8") (unit 1)
+        )
+      )
+    )
+  )
   (symbol (lib_id "Device:C") (at 52.07 132.08 180) (unit 1)
     (in_bom yes) (on_board yes) (dnp no)
@@
       (effects (font (size 1.27 1.27)))
     )
-    (property "Value" "DRV8212" (at 83.82 110.49 0)
-      (effects (font (size 1.27 1.27)))
-    )
+    (property "Value" "DRV8212DSG" (at 83.82 110.49 0)
+      (effects (font (size 1.27 1.27)))
+    )
